Commit message: added and tested lizi_description

File: lizi_description/urdf/lizi.urdf (robot description, URDF)
Before this commit: robot robotican_lizi.SLDASM, 12 links, 11 joints
Links:
- removed link FL_wheel_link
- removed link FR_wheel_link
- removed link RL_wheel_link
- removed link RR_wheel_link
- added link front_left_wheel_link, mass 0.201564744790293; collision mesh filename=package://lizi_description/meshes/front_left_wheel_link.STL; visual mesh filename=package://lizi_description/meshes/front_left_wheel_link.STL
- added link front_right_wheel_link, mass 0.201564744855459; collision mesh filename=package://lizi_description/meshes/front_right_wheel_link.STL; visual mesh filename=package://lizi_description/meshes/front_right_wheel_link.STL
- added link rear_left_wheel_link, mass 0.201564744787106; collision mesh filename=package://lizi_description/meshes/rear_left_wheel_link.STL; visual mesh filename=package://lizi_description/meshes/rear_left_wheel_link.STL
- added link rear_right_wheel_link, mass 0.201564744852236; collision mesh filename=package://lizi_description/meshes/rear_right_wheel_link.STL; visual mesh filename=package://lizi_description/meshes/rear_right_wheel_link.STL
- link base_link: geometry collision mesh filename=package://lizi_description/meshes/base_link.STL; visual mesh filename=package://lizi_description/meshes/base_link.STL
- link depth_cam_link: geometry collision mesh filename=package://lizi_description/meshes/depth_cam_link.STL; visual mesh filename=package://lizi_description/meshes/depth_cam_link.STL
- link laser_link: geometry collision mesh filename=package://lizi_description/meshes/laser_link.STL; visual mesh filename=package://lizi_description/meshes/laser_link.STL
Joints:
- removed joint FL_wheel_joint
- removed joint FR_wheell_joint
- removed joint RL_wheel_joint
- removed joint RR_wheel_joint
- added joint front_left_wheel_joint: type continuous, parent base_link, child front_left_wheel_link, origin xyz=0.13 0.1332125 0 rpy=0 0 0, axis 0 0.999999999981052 0
- added joint front_right_wheel_joint: type continuous, parent base_link, child front_right_wheel_link, origin xyz=0.130001640097326 -0.1332125 0 rpy=0 0 0, axis 0 0.999999999981052 0
- added joint rear_left_wheel_joint: type continuous, parent base_link, child rear_left_wheel_link, origin xyz=-0.13 0.1332125 0 rpy=0 0 0, axis 0 0.999999999993684 0
- added joint rear_right_wheel_joint: type continuous, parent base_link, child rear_right_wheel_link, origin xyz=-0.13 -0.1332125 0 rpy=0 0 0, axis 0 0.999999999993684 0
