Commit message: lot of fixes

File: lizi_description/urdf/lizi_gazebo.xacro (robot description, xacro)
@@ -49,117 +49,127 @@
     </xacro:if>
     <xacro:if value="$(arg urf)">
-        <xacro:urf name="left" link="left_urf_link" topic="URF/left" fov="${10.0*M_PI/180.0}" min="0.2" max="5.0"/>
-        <xacro:urf name="right" link="right_urf_link" topic="URF/right" fov="${10.0*M_PI/180.0}" min="0.2" max="5.0"/>
-        <xacro:urf name="rear" link="rear_urf_link" topic="URF/rear" fov="${10.0*M_PI/180.0}" min="0.2" max="5.0"/>
+        <xacro:urf name="left" link="left_urf_link" topic="urf/left" fov="${10.0*M_PI/180.0}" min="0.3" max="5.0" update_rate="10"/>
+        <xacro:urf name="right" link="right_urf_link" topic="urf/right" fov="${10.0*M_PI/180.0}" min="0.3" max="5.0" update_rate="10"/>
+        <xacro:urf name="rear" link="rear_urf_link" topic="urf/rear" fov="${10.0*M_PI/180.0}" min="0.3" max="5.0" update_rate="10"/>
     </xacro:if>
-        <xacro:if value="$(arg lidar)">
-            <xacro:lidar link="laser_link" topic="scan" samples="720" resolution="1" min_angle="-1.5707" max_angle="1.5707" range_min="0.1" range_max="30.0" range_resolution="0.01" />
-        </xacro:if>
-        <xacro:if value="$(arg gps)">
-            <xacro:gps link="base_link" hz="5" topic="GPS" lat="31.262218" long="34.80146100" alt="298"/>
-        </xacro:if>
-        <xacro:if value="$(arg imu)">
-            <xacro:imu link="base_link" hz="50" topic="IMU" />
-        </xacro:if>
-            <!-- controller manager and hardware interfaces -->
-            <xacro:if value="$(arg controllers)">
-                <gazebo>
-                    <plugin name="gazebo_ros_control" filename="libgazebo_ros_control.so">
-                        <robotSimType>gazebo_ros_control/DefaultRobotHWSim</robotSimType>
-                    </plugin>
-                </gazebo>
-                <!-- joints -->
-                <transmission name="front_left_wheel_joint_trans">
-                    <type>transmission_interface/SimpleTransmission</type>
-                    <joint name="front_left_wheel_joint">
-                        <hardwareInterface>hardware_interface/VelocityJointInterface</hardwareInterface>
-                    </joint>
-                    <actuator name="front_left_wheel_joint_motor">
-                        <mechanicalReduction>1</mechanicalReduction>
-                    </actuator>
-                </transmission>
-                <transmission name="front_right_wheel_joint_trans">
-                    <type>transmission_interface/SimpleTransmission</type>
-                    <joint name="front_right_wheel_joint">
-                        <hardwareInterface>hardware_interface/VelocityJointInterface</hardwareInterface>
-                    </joint>
-                    <actuator name="front_right_wheel_joint_motor">
-                        <mechanicalReduction>1</mechanicalReduction>
-                    </actuator>
-                </transmission>
-                <transmission name="rear_left_wheel_joint_trans">
-                    <type>transmission_interface/SimpleTransmission</type>
-                    <joint name="rear_left_wheel_joint">
-                        <hardwareInterface>hardware_interface/VelocityJointInterface</hardwareInterface>
-                    </joint>
-                    <actuator name="rear_left_wheel_joint_motor">
-                        <mechanicalReduction>1</mechanicalReduction>
-                    </actuator>
-                </transmission>
-                <transmission name="rear_right_wheel_joint_trans">
-                    <type>transmission_interface/SimpleTransmission</type>
-                    <joint name="rear_right_wheel_joint">
-                        <hardwareInterface>hardware_interface/VelocityJointInterface</hardwareInterface>
-                    </joint>
-                    <actuator name="rear_right_wheel_joint_motor">
-                        <mechanicalReduction>1</mechanicalReduction>
-                    </actuator>
-                </transmission>
-            </xacro:if>
-            <gazebo reference="front_left_wheel_link">
-                <!-- kp and kd for rubber -->
-               <kp>1000000.0</kp>
-                <kd>100.0</kd>
-                <mu1>1.5</mu1>
-                <mu2>1.5</mu2>
-                <fdir1>1 0 0</fdir1>
-                <maxVel>1.0</maxVel>
-                <minDepth>0.00</minDepth>
+    <xacro:if value="$(arg lidar)">
+        <xacro:lidar name="lidar"
+                     link="laser_link"
+                     topic="scan"
+                     update_rate="10"
+                     samples="720"
+                     resolution="1"
+                     min_angle="-1.5707"
+                     max_angle="1.5707"
+                     range_min="0.1"
+                     range_max="30.0"
+                     range_resolution="0.01" />
+    </xacro:if>
+    <xacro:if value="$(arg gps)">
+        <xacro:gps link="base_link" hz="5" topic="gps" lat="31.262218" long="34.80146100" alt="298"/>
+    </xacro:if>
+    <xacro:if value="$(arg imu)">
+        <xacro:imu link="base_link" hz="50" topic="imu" />
+    </xacro:if>
+    <!-- controller manager and hardware interfaces -->
+    <xacro:if value="$(arg controllers)">
+        <gazebo>
+            <plugin name="gazebo_ros_control" filename="libgazebo_ros_control.so">
+                <robotSimType>gazebo_ros_control/DefaultRobotHWSim</robotSimType>
+            </plugin>
+        </gazebo>
+        <!-- joints -->
+        <transmission name="front_left_wheel_joint_trans">
+            <type>transmission_interface/SimpleTransmission</type>
+            <joint name="front_left_wheel_joint">
+                <hardwareInterface>hardware_interface/VelocityJointInterface</hardwareInterface>
+            </joint>
+            <actuator name="front_left_wheel_joint_motor">
+                <mechanicalReduction>1</mechanicalReduction>
+            </actuator>
+        </transmission>
+        <transmission name="front_right_wheel_joint_trans">
+            <type>transmission_interface/SimpleTransmission</type>
+            <joint name="front_right_wheel_joint">
+                <hardwareInterface>hardware_interface/VelocityJointInterface</hardwareInterface>
+            </joint>
+            <actuator name="front_right_wheel_joint_motor">
+                <mechanicalReduction>1</mechanicalReduction>
+            </actuator>
+        </transmission>
+        <transmission name="rear_left_wheel_joint_trans">
+            <type>transmission_interface/SimpleTransmission</type>
+            <joint name="rear_left_wheel_joint">
+                <hardwareInterface>hardware_interface/VelocityJointInterface</hardwareInterface>
+            </joint>
+            <actuator name="rear_left_wheel_joint_motor">
+                <mechanicalReduction>1</mechanicalReduction>
+            </actuator>
+        </transmission>
+        <transmission name="rear_right_wheel_joint_trans">
+            <type>transmission_interface/SimpleTransmission</type>
+            <joint name="rear_right_wheel_joint">
+                <hardwareInterface>hardware_interface/VelocityJointInterface</hardwareInterface>
+            </joint>
+            <actuator name="rear_right_wheel_joint_motor">
+                <mechanicalReduction>1</mechanicalReduction>
+            </actuator>
+        </transmission>
+    </xacro:if>
+    <gazebo reference="front_left_wheel_link">
+        <!-- kp and kd for rubber -->
+        <kp>1000000.0</kp>
+        <kd>100.0</kd>
+        <mu1>1.5</mu1>
+        <mu2>1.5</mu2>
+        <fdir1>1 0 0</fdir1>
+        <maxVel>1.0</maxVel>
+        <minDepth>0.00</minDepth>
 <!--                <material>Gazebo/Black</material>-->
-            </gazebo>
-            <gazebo reference="front_right_wheel_link">
-              <!-- kp and kd for rubber -->
-              <kp>1000000.0</kp>
-                <kd>100.0</kd>
-                <mu1>1.5</mu1>
-                <mu2>1.5</mu2>
-                <fdir1>1 0 0</fdir1>
-                <maxVel>1.0</maxVel>
-                <minDepth>0.00</minDepth>
+    </gazebo>
+    <gazebo reference="front_right_wheel_link">
+        <!-- kp and kd for rubber -->
+        <kp>1000000.0</kp>
+        <kd>100.0</kd>
+        <mu1>1.5</mu1>
+        <mu2>1.5</mu2>
+        <fdir1>1 0 0</fdir1>
+        <maxVel>1.0</maxVel>
+        <minDepth>0.00</minDepth>
 <!--                <material>Gazebo/Black</material>-->
-            </gazebo>
-            <gazebo reference="rear_left_wheel_link">
-               <!-- kp and kd for rubber -->
-              <kp>1000000.0</kp>
-                <kd>100.0</kd>
-                <mu1>1.5</mu1>
-                <mu2>1.5</mu2>
-                <fdir1>1 0 0</fdir1>
-                <maxVel>1.0</maxVel>
-                <minDepth>0.00</minDepth>
+    </gazebo>
+    <gazebo reference="rear_left_wheel_link">
+        <!-- kp and kd for rubber -->
+        <kp>1000000.0</kp>
+        <kd>100.0</kd>
+        <mu1>1.5</mu1>
+        <mu2>1.5</mu2>
+        <fdir1>1 0 0</fdir1>
+        <maxVel>1.0</maxVel>
+        <minDepth>0.00</minDepth>
 <!--                <material>Gazebo/Black</material>-->
-            </gazebo>
-            <gazebo reference="rear_right_wheel_link">
-           <!-- kp and kd for rubber -->
-               <kp>1000000.0</kp>
-                <kd>100.0</kd>
-                <mu1>1.5</mu1>
-                <mu2>1.5</mu2>
-                <fdir1>1 0 0</fdir1>
-                <maxVel>1.0</maxVel>
-                <minDepth>0.00</minDepth>
+    </gazebo>
+    <gazebo reference="rear_right_wheel_link">
+    <!-- kp and kd for rubber -->
+        <kp>1000000.0</kp>
+        <kd>100.0</kd>
+        <mu1>1.5</mu1>
+        <mu2>1.5</mu2>
+        <fdir1>1 0 0</fdir1>
+        <maxVel>1.0</maxVel>
+        <minDepth>0.00</minDepth>
 <!--                <material>Gazebo/Black</material>-->
-            </gazebo>
-            <gazebo reference="base_link">
-                <material>Gazebo/Grey</material>
-            </gazebo>
-            <gazebo reference="left_urf_link">
-                <material>Gazebo/Black</material>
-            </gazebo>
-            <gazebo reference="rear_urf_link">
-                <material>Gazebo/Black</material>
-            </gazebo>
-            <gazebo reference="right_urf_link">
-                <material>Gazebo/Black</material>
-            </gazebo>
-        </robot>
+    </gazebo>
+    <gazebo reference="base_link">
+        <material>Gazebo/Grey</material>
+    </gazebo>
+    <gazebo reference="left_urf_link">
+        <material>Gazebo/Black</material>
+    </gazebo>
+    <gazebo reference="rear_urf_link">
+        <material>Gazebo/Black</material>
+    </gazebo>
+    <gazebo reference="right_urf_link">
+        <material>Gazebo/Black</material>
+    </gazebo>
+</robot>
