Commit message: added cam macro

File: lizi_description/urdf/lizi.xacro (robot description, xacro)
@@ -24,19 +24,19 @@
       <geometry>
         <mesh
-          filename="package://lizi_description/meshes/base_link.STL" />
-      </geometry>
-      <material
-        name="">
-        <color
-          rgba="0.792156862745098 0.819607843137255 0.933333333333333 1" />
-      </material>
-    </visual>
-    <collision>
-      <origin
-        xyz="0 0 0"
-        rpy="0 0 0" />
-      <geometry>
-        <mesh
-          filename="package://lizi_description/meshes/base_link.STL" />
+          filename="package://lizi_description/meshes/base.STL" />
+      </geometry>
+      <material
+        name="">
+        <color
+          rgba="0.792156862745098 0.819607843137255 0.933333333333333 1" />
+      </material>
+    </visual>
+    <collision>
+      <origin
+        xyz="0 0 0"
+        rpy="0 0 0" />
+      <geometry>
+        <mesh
+          filename="package://lizi_description/meshes/base.STL" />
       </geometry>
     </collision>
@@ -79,5 +79,5 @@
       <geometry>
         <mesh
-          filename="package://lizi_description/meshes/laser_link.STL" />
+          filename="package://lizi_description/meshes/lidar.STL" />
       </geometry>
       <material
@@ -93,5 +93,5 @@
       <geometry>
         <mesh
-          filename="package://lizi_description/meshes/laser_link.STL" />
+          filename="package://lizi_description/meshes/lidar.STL" />
       </geometry>
     </collision>
@@ -132,19 +132,19 @@
       <geometry>
         <mesh
-          filename="package://lizi_description/meshes/depth_cam_link.STL" />
-      </geometry>
-      <material
-        name="">
-        <color
-          rgba="0.792156862745098 0.819607843137255 0.933333333333333 1" />
-      </material>
-    </visual>
-    <collision>
-      <origin
-        xyz="0 0 0"
-        rpy="0 0 0" />
-      <geometry>
-        <mesh
-          filename="package://lizi_description/meshes/depth_cam_link.STL" />
+          filename="package://lizi_description/meshes/depth_cam.STL" />
+      </geometry>
+      <material
+        name="">
+        <color
+          rgba="0.792156862745098 0.819607843137255 0.933333333333333 1" />
+      </material>
+    </visual>
+    <collision>
+      <origin
+        xyz="0 0 0"
+        rpy="0 0 0" />
+      <geometry>
+        <mesh
+          filename="package://lizi_description/meshes/depth_cam.STL" />
       </geometry>
     </collision>
@@ -230,19 +230,19 @@
       <geometry>
         <mesh
-          filename="package://lizi_description/meshes/front_left_wheel_link.STL" />
-      </geometry>
-      <material
-        name="">
-        <color
-          rgba="0.792156862745098 0.819607843137255 0.933333333333333 1" />
-      </material>
-    </visual>
-    <collision>
-      <origin
-        xyz="0 0 0"
-        rpy="0 0 0" />
-      <geometry>
-        <mesh
-          filename="package://lizi_description/meshes/front_left_wheel_link.STL" />
+          filename="package://lizi_description/meshes/wheel.STL" />
+      </geometry>
+      <material
+        name="">
+        <color
+          rgba="0.792156862745098 0.819607843137255 0.933333333333333 1" />
+      </material>
+    </visual>
+    <collision>
+      <origin
+        xyz="0 0 0"
+        rpy="0 0 0" />
+      <geometry>
+        <mesh
+          filename="package://lizi_description/meshes/wheel.STL" />
       </geometry>
     </collision>
@@ -283,19 +283,19 @@
       <geometry>
         <mesh
-          filename="package://lizi_description/meshes/rear_left_wheel_link.STL" />
-      </geometry>
-      <material
-        name="">
-        <color
-          rgba="0.792156862745098 0.819607843137255 0.933333333333333 1" />
-      </material>
-    </visual>
-    <collision>
-      <origin
-        xyz="0 0 0"
-        rpy="0 0 0" />
-      <geometry>
-        <mesh
-          filename="package://lizi_description/meshes/rear_left_wheel_link.STL" />
+          filename="package://lizi_description/meshes/wheel.STL" />
+      </geometry>
+      <material
+        name="">
+        <color
+          rgba="0.792156862745098 0.819607843137255 0.933333333333333 1" />
+      </material>
+    </visual>
+    <collision>
+      <origin
+        xyz="0 0 0"
+        rpy="0 0 0" />
+      <geometry>
+        <mesh
+          filename="package://lizi_description/meshes/wheel.STL" />
       </geometry>
     </collision>
@@ -336,19 +336,19 @@
       <geometry>
         <mesh
-          filename="package://lizi_description/meshes/front_right_wheel_link.STL" />
-      </geometry>
-      <material
-        name="">
-        <color
-          rgba="0.792156862745098 0.819607843137255 0.933333333333333 1" />
-      </material>
-    </visual>
-    <collision>
-      <origin
-        xyz="0 0 0"
-        rpy="0 0 0" />
-      <geometry>
-        <mesh
-          filename="package://lizi_description/meshes/front_right_wheel_link.STL" />
+          filename="package://lizi_description/meshes/wheel.STL" />
+      </geometry>
+      <material
+        name="">
+        <color
+          rgba="0.792156862745098 0.819607843137255 0.933333333333333 1" />
+      </material>
+    </visual>
+    <collision>
+      <origin
+        xyz="0 0 0"
+        rpy="0 0 0" />
+      <geometry>
+        <mesh
+          filename="package://lizi_description/meshes/wheel.STL" />
       </geometry>
     </collision>
@@ -389,19 +389,19 @@
       <geometry>
         <mesh
-          filename="package://lizi_description/meshes/rear_right_wheel_link.STL" />
-      </geometry>
-      <material
-        name="">
-        <color
-          rgba="0.792156862745098 0.819607843137255 0.933333333333333 1" />
-      </material>
-    </visual>
-    <collision>
-      <origin
-        xyz="0 0 0"
-        rpy="0 0 0" />
-      <geometry>
-        <mesh
-          filename="package://lizi_description/meshes/rear_right_wheel_link.STL" />
+          filename="package://lizi_description/meshes/wheel.STL" />
+      </geometry>
+      <material
+        name="">
+        <color
+          rgba="0.792156862745098 0.819607843137255 0.933333333333333 1" />
+      </material>
+    </visual>
+    <collision>
+      <origin
+        xyz="0 0 0"
+        rpy="0 0 0" />
+      <geometry>
+        <mesh
+          filename="package://lizi_description/meshes/wheel.STL" />
       </geometry>
     </collision>
@@ -421,7 +421,7 @@
   </joint>
   <link
-    name="front_camera_link" />
-  <joint
-    name="front_camera_joint"
+    name="cam_link" />
+  <joint
+    name="cam_joint"
     type="fixed">
     <origin
@@ -431,5 +431,5 @@
       link="base_link" />
     <child
-      link="front_camera_link" />
+      link="cam_link" />
     <axis
       xyz="0 0 0" />

File: lizi_description/urdf/lizi_gazebo.xacro (robot description, xacro)
@@ -2,5 +2,10 @@
 <robot xmlns:xacro="http://www.ros.org/wiki/xacro" name="lizi" description="Lizi robot">
     <xacro:include filename="$(find lizi_description)/urdf/lizi.xacro" />
-    <xacro:include filename="$(find mobilican_macros)/camera.xacro" />
+    <xacro:include filename="$(find mobilican_macros)/macros/depth_cam.xacro" />
+    <xacro:include filename="$(find mobilican_macros)/macros/cam.xacro" />
+    <xacro:include filename="$(find mobilican_macros)/macros/urf.xacro" />
+    <xacro:include filename="$(find mobilican_macros)/macros/lidar.xacro" />
+    <xacro:include filename="$(find mobilican_macros)/macros/gps.xacro" />
+    <xacro:include filename="$(find mobilican_macros)/macros/imu.xacro" />
     <xacro:property name="M_PI" value="3.14159265358979" />
     <xacro:property name="URF_FOV" value="${10.0*M_PI/180}" />
@@ -10,35 +15,48 @@
     <xacro:arg name="gps" default="false"/>
     <xacro:arg name="lidar" default="false"/>
-    <xacro:arg name="rgb_cam" default="false"/>
+    <xacro:arg name="cam" default="false"/>
     <xacro:arg name="depth_cam" default="false"/>
-    <!-- cameras  -->
-    <xacro:if value="$(arg rgb_cam)">
-        <xacro:Camera name="rgb_cam" link="rgb_cam_link" image_width="640" image_height="480"
-                      image_format="R8G8B8" clip_near="0.02" clip_far="300" />
-        </xacro:if>
-        <xacro:if value="$(arg depth_cam)">
-           <xacro:include filename="$(find mobilican_macros)/depth_cam.xacro" />
-           <xacro:softkinetic_gazebo name="softkinetic_rgb" ros_topic="softkinetic"/>
-        </xacro:if>
-        <!-- Sonars -->
-        <xacro:if value="$(arg urf)">
-            <xacro:include filename="$(find mobilican_macros)/urf.xacro" />
-            <xacro:urf name="left" link="left_urf_link" topic="URF/left" fov="${10.0*M_PI/180.0}" min="0.2" max="5.0"/>
-            <xacro:urf name="right" link="right_urf_link" topic="URF/right" fov="${10.0*M_PI/180.0}" min="0.2" max="5.0"/>
-            <xacro:urf name="rear" link="rear_urf_link" topic="URF/rear" fov="${10.0*M_PI/180.0}" min="0.2" max="5.0"/>
-        </xacro:if>
-        <!-- hokuyo -->
+   <xacro:if value="$(arg cam)">
+        <xacro:Camera name="camera"
+                      link="cam_link"
+                      image_width="1280"
+                      image_height="720"
+                      image_format="R8G8B8"
+                      clip_near="0.02"
+                      clip_far="200"
+                      image_topic="image_raw"
+                      info_topic="info"
+                      update_rate="30"
+                      horizontal_fov="1.064" />
+    </xacro:if>
+    <xacro:if value="$(arg depth_cam)">
+        <xacro:DepthCam name="depth_cam"
+                        link="depth_cam_link"
+                        horizontal_fov="1.592"
+                        img_width="1280"
+                        img_height="800"
+                        img_format="B8G8R8"
+                        clip_near="0.1"
+                        clip_far="200"
+                        update_rate="30.0"
+                        image_topic="color/image_raw"
+                        depth_topic="depth/color/image_raw"
+                        cloud_topic="depth/color/points"
+                        info_topic="color/camera_info"
+                        depth_info_topic="depth/camera_info"
+                        pointcloud_cuttoff="0.2" />
+    </xacro:if>
+    <xacro:if value="$(arg urf)">
+        <xacro:urf name="left" link="left_urf_link" topic="URF/left" fov="${10.0*M_PI/180.0}" min="0.2" max="5.0"/>
+        <xacro:urf name="right" link="right_urf_link" topic="URF/right" fov="${10.0*M_PI/180.0}" min="0.2" max="5.0"/>
+        <xacro:urf name="rear" link="rear_urf_link" topic="URF/rear" fov="${10.0*M_PI/180.0}" min="0.2" max="5.0"/>
+    </xacro:if>
         <xacro:if value="$(arg lidar)">
-            <xacro:include filename="$(find mobilican_macros)/hokuyo.xacro" />
             <xacro:lidar link="laser_link" topic="scan" samples="720" resolution="1" min_angle="-1.5707" max_angle="1.5707" range_min="0.1" range_max="30.0" range_resolution="0.01" />
         </xacro:if>
-        <!-- GPS   -->
         <xacro:if value="$(arg gps)">
-            <xacro:include filename="$(find mobilican_macros)/gps.xacro" />
             <xacro:gps link="base_link" hz="5" topic="GPS" lat="31.262218" long="34.80146100" alt="298"/>
         </xacro:if>
-        <!-- IMU   -->
         <xacro:if value="$(arg imu)">
-            <xacro:include filename="$(find mobilican_macros)/imu.xacro" />
             <xacro:imu link="base_link" hz="50" topic="IMU" />
         </xacro:if>

Commit message: fixed deattached base footprint

File: lizi_description/urdf/lizi.xacro (robot description, xacro)
@@ -1,5 +1,6 @@
 <?xml version="1.0" encoding="UTF-8"?>
 <robot
-  name="lizi">
+  xmlns:xacro="http://www.ros.org/wiki/xacro" name="lizi">
+  <xacro:property name="M_PI" value="3.14159265358979" />
   <link
     name="base_link">
@@ -43,7 +44,7 @@
   </link>
   <link
-    name="footprint_link" />
-  <joint
-    name="footprint_joint"
+    name="base_footprint" />
+  <joint
+    name="base_footprint_joint"
     type="fixed">
     <origin
@@ -51,7 +52,7 @@
       rpy="0 0 0" />
     <parent
-      link="base_link" />
-    <child
-      link="footprint_link" />
+      link="base_footprint" />
+    <child
+      link="base_link" />
     <axis
       xyz="0 0 0" />
@@ -435,3 +436,55 @@
       xyz="0 0 0" />
   </joint>
+      <!-- camera depth joints and links -->
+    <joint name="camera_depth_joint" type="fixed">
+      <origin xyz="0 -0.0122 0" rpy="0 0 0"/>
+      <parent link="depth_cam_link"/>
+      <child link="camera_depth_frame" />
+    </joint>
+    <link name="camera_depth_frame"/>
+    <joint name="camera_depth_optical_joint" type="fixed">
+      <origin xyz="0 0 0" rpy="${-M_PI/2} 0 ${-M_PI/2}" />
+      <parent link="camera_depth_frame" />
+      <child link="camera_depth_optical_frame" />
+    </joint>
+    <link name="camera_depth_optical_frame"/>
+    <!-- camera left IR joints and links -->
+    <joint name="camera_left_ir_joint" type="fixed">
+      <origin xyz="0 -0.0322 0" rpy="0 0 0" />
+      <parent link="depth_cam_link" />
+      <child link="camera_left_ir_frame" />
+    </joint>
+    <link name="camera_left_ir_frame"/>
+    <joint name="camera_left_ir_optical_joint" type="fixed">
+      <origin xyz="0 0 0" rpy="${-M_PI/2} 0 ${-M_PI/2}" />
+      <parent link="camera_left_ir_frame" />
+      <child link="camera_left_ir_optical_frame" />
+    </joint>
+    <link name="camera_left_ir_optical_frame"/>
+    <!-- camera right IR joints and links -->
+    <joint name="camera_right_ir_joint" type="fixed">
+      <origin xyz="0 0.0178 0" rpy="0 0 0" />
+      <parent link="depth_cam_link" />
+      <child link="camera_right_ir_frame" />
+    </joint>
+    <link name="camera_right_ir_frame"/>
+    <joint name="camera_right_ir_optical_joint" type="fixed">
+      <origin xyz="0 0 0" rpy="${-M_PI/2} 0 ${-M_PI/2}" />
+      <parent link="camera_right_ir_frame" />
+      <child link="camera_right_ir_optical_frame" />
+    </joint>
+    <link name="camera_right_ir_optical_frame"/>
+    <!-- camera fisheye joints and links -->
+    <joint name="camera_fisheye_joint" type="fixed">
+      <origin xyz="0 0.0322 0" rpy="0 0 0" />
+      <parent link="depth_cam_link" />
+      <child link="camera_fisheye_frame" />
+    </joint>
+    <link name="camera_fisheye_frame"/>
+    <joint name="camera_fisheye_optical_joint" type="fixed">
+      <origin xyz="0 0 0" rpy="${-M_PI/2} 0 ${-M_PI/2}" />
+      <parent link="camera_fisheye_frame" />
+      <child link="camera_fisheye_optical_frame" />
+    </joint>
+    <link name="camera_fisheye_optical_frame"/>
 </robot>

File: lizi_description/urdf/lizi_gazebo.xacro (robot description, xacro)
@@ -33,4 +33,5 @@
         <xacro:DepthCam name="depth_cam"
                         link="depth_cam_link"
+                        optical_frame="camera_depth_optical_frame"
                         horizontal_fov="1.592"
                         img_width="1280"

Commit message: added d435 launch. tested ok

File: lizi_description/urdf/lizi.xacro (robot description, xacro)
@@ -112,5 +112,5 @@
   </joint>
   <link
-    name="depth_cam_link">
+    name="camera_link">
     <inertial>
       <origin
@@ -160,5 +160,5 @@
       link="base_link" />
     <child
-      link="depth_cam_link" />
+      link="camera_link" />
     <axis
       xyz="0 0 0" />
@@ -422,5 +422,5 @@
   </joint>
   <link
-    name="cam_link" />
+    name="rgb_cam_link" />
   <joint
     name="cam_joint"
@@ -432,5 +432,5 @@
       link="base_link" />
     <child
-      link="cam_link" />
+      link="rgb_cam_link" />
     <axis
       xyz="0 0 0" />
@@ -439,5 +439,5 @@
     <joint name="camera_depth_joint" type="fixed">
       <origin xyz="0 -0.0122 0" rpy="0 0 0"/>
-      <parent link="depth_cam_link"/>
+      <parent link="camera_link"/>
       <child link="camera_depth_frame" />
     </joint>
@@ -452,5 +452,5 @@
     <joint name="camera_left_ir_joint" type="fixed">
       <origin xyz="0 -0.0322 0" rpy="0 0 0" />
-      <parent link="depth_cam_link" />
+      <parent link="camera_link" />
       <child link="camera_left_ir_frame" />
     </joint>
@@ -465,5 +465,5 @@
     <joint name="camera_right_ir_joint" type="fixed">
       <origin xyz="0 0.0178 0" rpy="0 0 0" />
-      <parent link="depth_cam_link" />
+      <parent link="camera_link" />
       <child link="camera_right_ir_frame" />
     </joint>
@@ -478,5 +478,5 @@
     <joint name="camera_fisheye_joint" type="fixed">
       <origin xyz="0 0.0322 0" rpy="0 0 0" />
-      <parent link="depth_cam_link" />
+      <parent link="camera_link" />
       <child link="camera_fisheye_frame" />
     </joint>

Commit message: reduce wheels friction in gazebo

File: lizi_description/urdf/lizi.xacro (robot description, xacro)
@@ -10,5 +10,5 @@
         rpy="0 0 0" />
       <mass
-        value="0.470251986966204" />
+        value="3.470251986966204" />
       <inertia
         ixx="0.00417603662557191"

File: lizi_description/urdf/lizi_gazebo.xacro (robot description, xacro)
@@ -117,10 +117,12 @@
         </transmission>
     </xacro:if>
+    <xacro:property name="mu1" value="1.0" />
+    <xacro:property name="mu2" value="1.0" />
     <gazebo reference="front_left_wheel_link">
         <!-- kp and kd for rubber -->
         <kp>1000000.0</kp>
         <kd>100.0</kd>
-        <mu1>1.5</mu1>
-        <mu2>1.5</mu2>
+        <mu1>${mu1}</mu1>
+        <mu2>${mu2}</mu2>
         <fdir1>1 0 0</fdir1>
         <maxVel>1.0</maxVel>
@@ -132,6 +134,6 @@
         <kp>1000000.0</kp>
         <kd>100.0</kd>
-        <mu1>1.5</mu1>
-        <mu2>1.5</mu2>
+        <mu1>${mu1}</mu1>
+        <mu2>${mu2}</mu2>
         <fdir1>1 0 0</fdir1>
         <maxVel>1.0</maxVel>
@@ -143,6 +145,6 @@
         <kp>1000000.0</kp>
         <kd>100.0</kd>
-        <mu1>1.5</mu1>
-        <mu2>1.5</mu2>
+        <mu1>${mu1}</mu1>
+        <mu2>${mu2}</mu2>
         <fdir1>1 0 0</fdir1>
         <maxVel>1.0</maxVel>
@@ -154,6 +156,6 @@
         <kp>1000000.0</kp>
         <kd>100.0</kd>
-        <mu1>1.5</mu1>
-        <mu2>1.5</mu2>
+        <mu1>${mu1}</mu1>
+        <mu2>${mu2}</mu2>
         <fdir1>1 0 0</fdir1>
         <maxVel>1.0</maxVel>

Commit message: added installations to setup script

File: lizi_description/urdf/lizi.xacro (robot description, xacro)
@@ -7,8 +7,8 @@
     <inertial>
       <origin
-        xyz="0.00417829000094622 0.00524236473615063 0.0404695921883583"
-        rpy="0 0 0" />
-      <mass
-        value="3.470251986966204" />
+        xyz="6.00417829000094622 0.00524236473615063 0.0404695921883583"
+        rpy="0 0 0" />
+      <mass
+        value="0.170251986966204" />
       <inertia
         ixx="0.00417603662557191"

Commit message: fixed inertia in sim

File: lizi_description/urdf/lizi.xacro (robot description, xacro)
@@ -7,8 +7,8 @@
     <inertial>
       <origin
-        xyz="6.00417829000094622 0.00524236473615063 0.0404695921883583"
-        rpy="0 0 0" />
-      <mass
-        value="0.170251986966204" />
+        xyz="0.0030152 0.00524236473615063 0.0404695921883583"
+        rpy="0 0 0" />
+      <mass
+        value="1.170251986966204" />
       <inertia
         ixx="0.00417603662557191"
@@ -242,8 +242,7 @@
       <origin
         xyz="0 0 0"
-        rpy="0 0 0" />
-      <geometry>
-        <mesh
-          filename="package://lizi_description/meshes/wheel.STL" />
+        rpy="${M_PI/2} 0 0" />
+      <geometry>
+        <cylinder  length="0.025" radius="0.076"/>
       </geometry>
     </collision>
@@ -295,8 +294,7 @@
       <origin
         xyz="0 0 0"
-        rpy="0 0 0" />
-      <geometry>
-        <mesh
-          filename="package://lizi_description/meshes/wheel.STL" />
+        rpy="${M_PI/2} 0 0" />
+      <geometry>
+        <cylinder  length="0.025" radius="0.076"/>
       </geometry>
     </collision>
@@ -348,8 +346,7 @@
       <origin
         xyz="0 0 0"
-        rpy="0 0 0" />
-      <geometry>
-        <mesh
-          filename="package://lizi_description/meshes/wheel.STL" />
+        rpy="${M_PI/2} 0 0" />
+      <geometry>
+        <cylinder  length="0.025" radius="0.076"/>
       </geometry>
     </collision>
@@ -401,8 +398,7 @@
       <origin
         xyz="0 0 0"
-        rpy="0 0 0" />
-      <geometry>
-        <mesh
-          filename="package://lizi_description/meshes/wheel.STL" />
+        rpy="${M_PI/2} 0 0" />
+      <geometry>
+        <cylinder  length="0.025" radius="0.076"/>
       </geometry>
     </collision>

Commit message: added the right colors to the model

File: lizi_description/urdf/lizi.xacro (robot description, xacro)
@@ -10,5 +10,5 @@
         rpy="0 0 0" />
       <mass
-        value="1.170251986966204" />
+        value="5.470251986966204" />
       <inertia
         ixx="0.00417603662557191"
@@ -30,5 +30,5 @@
         name="">
         <color
-          rgba="0.792156862745098 0.819607843137255 0.933333333333333 1" />
+          rgba="0 0 0.8 1" />
       </material>
     </visual>

File: lizi_description/urdf/lizi_gazebo.xacro (robot description, xacro)
@@ -128,5 +128,5 @@
         <maxVel>1.0</maxVel>
         <minDepth>0.00</minDepth>
-<!--                <material>Gazebo/Black</material>-->
+        <material>Gazebo/DarkGrey</material>
     </gazebo>
     <gazebo reference="front_right_wheel_link">
@@ -139,5 +139,5 @@
         <maxVel>1.0</maxVel>
         <minDepth>0.00</minDepth>
-<!--                <material>Gazebo/Black</material>-->
+        <material>Gazebo/DarkGrey</material>
     </gazebo>
     <gazebo reference="rear_left_wheel_link">
@@ -150,5 +150,5 @@
         <maxVel>1.0</maxVel>
         <minDepth>0.00</minDepth>
-<!--                <material>Gazebo/Black</material>-->
+        <material>Gazebo/DarkGrey</material>
     </gazebo>
     <gazebo reference="rear_right_wheel_link">
@@ -161,8 +161,8 @@
         <maxVel>1.0</maxVel>
         <minDepth>0.00</minDepth>
-<!--                <material>Gazebo/Black</material>-->
+        <material>Gazebo/DarkGrey</material>
     </gazebo>
     <gazebo reference="base_link">
-        <material>Gazebo/Grey</material>
+        <material>Gazebo/Grass</material>
     </gazebo>
     <gazebo reference="left_urf_link">
@@ -175,3 +175,9 @@
         <material>Gazebo/Black</material>
     </gazebo>
+    <gazebo reference="laser_link">
+        <material>Gazebo/DarkGrey</material>
+    </gazebo>
+    <gazebo reference="camera_link">
+        <material>Gazebo/Grey</material>
+    </gazebo>
 </robot>
